Commit message: Rename robot description package

File: src/kiwi_description/kiwi_drive_description/urdf/Kiwi_Drive_Full_Assembly_Copy_Copy.urdf (robot description, URDF)
Before this commit: robot Kiwi_Drive_Full_Assembly_Copy_Copy, 5 links, 4 joints
Links:
- link Lidar_Mounting_Plate: geometry collision mesh filename=package://kiwi_drive_description/meshes/lidar_link/Lidar_Mo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 scale=0.01 0.01 0.01; visual mesh filename=package://kiwi_drive_description/meshes/lidar_link/Lidar_Mo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 scale=1 1 1
- link base_link: geometry collision mesh filename=package://kiwi_drive_description/meshes/base_link/base_link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 scale=0.01 0.01 0.01; visual mesh filename=package://kiwi_drive_description/meshes/base_link/base_link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 scale=1 1 1
- link wheel_1_link_Omni_Wheel: geometry collision mesh filename=package://kiwi_drive_description/meshes/wheel_1_link/wheel_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 scale=0.01 0.01 0.01; visual mesh filename=package://kiwi_drive_description/meshes/wheel_1_link/wheel_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 scale=1 1 1
- link wheel_2_link_Omni_Wheel: geometry collision mesh filename=package://kiwi_drive_description/meshes/wheel_2_link/wheel_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 scale=0.01 0.01 0.01; visual mesh filename=package://kiwi_drive_description/meshes/wheel_2_link/wheel_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 scale=1 1 1
- link wheel_3_link_Omni_Wheel: geometry collision mesh filename=package://kiwi_drive_description/meshes/wheel_3_link/wheel_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 scale=0.01 0.01 0.01; visual mesh filename=package://kiwi_drive_description/meshes/wheel_3_link/wheel_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 scale=1 1 1

File: src/kiwi_description/kiwi_drive_description/urdf/Kiwi_Drive_Full_Assembly_Copy_Copy.urdf.xacro (robot description, xacro)
@@ -6,9 +6,9 @@
   </material>
   <!-- Assembly includes -->
-  <xacro:include filename="$(find Kiwi_Drive_Full_Assembly_Copy_Copy_description)/urdf/assemblies/base_link.urdf.xacro"/>
-  <xacro:include filename="$(find Kiwi_Drive_Full_Assembly_Copy_Copy_description)/urdf/assemblies/wheel_1_link.urdf.xacro"/>
-  <xacro:include filename="$(find Kiwi_Drive_Full_Assembly_Copy_Copy_description)/urdf/assemblies/wheel_2_link.urdf.xacro"/>
-  <xacro:include filename="$(find Kiwi_Drive_Full_Assembly_Copy_Copy_description)/urdf/assemblies/wheel_3_link.urdf.xacro"/>
-  <xacro:include filename="$(find Kiwi_Drive_Full_Assembly_Copy_Copy_description)/urdf/assemblies/lidar_link.urdf.xacro"/>
+  <xacro:include filename="$(find kiwi_drive_description)/urdf/assemblies/base_link.urdf.xacro"/>
+  <xacro:include filename="$(find kiwi_drive_description)/urdf/assemblies/wheel_1_link.urdf.xacro"/>
+  <xacro:include filename="$(find kiwi_drive_description)/urdf/assemblies/wheel_2_link.urdf.xacro"/>
+  <xacro:include filename="$(find kiwi_drive_description)/urdf/assemblies/wheel_3_link.urdf.xacro"/>
+  <xacro:include filename="$(find kiwi_drive_description)/urdf/assemblies/lidar_link.urdf.xacro"/>
   <!-- Instantiate assemblies -->
   <xacro:base_link prefix=""/>

File: src/kiwi_description/kiwi_drive_description/urdf/assemblies/base_link.urdf.xacro (robot description, xacro)
@@ -13,5 +13,5 @@
         <origin xyz="0.000000 0.000000 0.000000" rpy="0.000000 0.000000 -2.094395"/>
         <geometry>
-          <mesh filename="package://Kiwi_Drive_Full_Assembly_Copy_Copy_description/meshes/base_link/base_link.dae" scale="1 1 1"/>
+          <mesh filename="package://kiwi_drive_description/meshes/base_link/base_link.dae" scale="1 1 1"/>
         </geometry>
         <material name="Steel"/>
@@ -20,5 +20,5 @@
         <origin xyz="0.000000 0.000000 0.000000" rpy="0.000000 0.000000 -2.094395"/>
         <geometry>
-          <mesh filename="package://Kiwi_Drive_Full_Assembly_Copy_Copy_description/meshes/base_link/base_link_collision.stl" scale="0.01 0.01 0.01"/>
+          <mesh filename="package://kiwi_drive_description/meshes/base_link/base_link_collision.stl" scale="0.01 0.01 0.01"/>
         </geometry>
       </collision>

File: src/kiwi_description/kiwi_drive_description/urdf/assemblies/lidar_link.urdf.xacro (robot description, xacro)
@@ -13,5 +13,5 @@
         <origin xyz="0.000000 0.000000 0.000000" rpy="0.000000 0.000000 0.000000"/>
         <geometry>
-          <mesh filename="package://Kiwi_Drive_Full_Assembly_Copy_Copy_description/meshes/lidar_link/Lidar_Mounting_Plate.dae" scale="1 1 1"/>
+          <mesh filename="package://kiwi_drive_description/meshes/lidar_link/Lidar_Mounting_Plate.dae" scale="1 1 1"/>
         </geometry>
         <material name="Steel"/>
@@ -20,5 +20,5 @@
         <origin xyz="0.000000 0.000000 0.000000" rpy="0.000000 0.000000 0.000000"/>
         <geometry>
-          <mesh filename="package://Kiwi_Drive_Full_Assembly_Copy_Copy_description/meshes/lidar_link/Lidar_Mounting_Plate_collision.stl" scale="0.01 0.01 0.01"/>
+          <mesh filename="package://kiwi_drive_description/meshes/lidar_link/Lidar_Mounting_Plate_collision.stl" scale="0.01 0.01 0.01"/>
         </geometry>
       </collision>

File: src/kiwi_description/kiwi_drive_description/urdf/assemblies/wheel_1_link.urdf.xacro (robot description, xacro)
@@ -13,5 +13,5 @@
         <origin xyz="-0.088814 0.603225 0.367959" rpy="3.119159 -1.068867 -1.590625"/>
         <geometry>
-          <mesh filename="package://Kiwi_Drive_Full_Assembly_Copy_Copy_description/meshes/wheel_1_link/wheel_1_link_Omni_Wheel.dae" scale="1 1 1"/>
+          <mesh filename="package://kiwi_drive_description/meshes/wheel_1_link/wheel_1_link_Omni_Wheel.dae" scale="1 1 1"/>
         </geometry>
         <material name="Steel"/>
@@ -20,5 +20,5 @@
         <origin xyz="-0.088814 0.603225 0.367959" rpy="3.119159 -1.068867 -1.590625"/>
         <geometry>
-          <mesh filename="package://Kiwi_Drive_Full_Assembly_Copy_Copy_description/meshes/wheel_1_link/wheel_1_link_Omni_Wheel_collision.stl" scale="0.01 0.01 0.01"/>
+          <mesh filename="package://kiwi_drive_description/meshes/wheel_1_link/wheel_1_link_Omni_Wheel_collision.stl" scale="0.01 0.01 0.01"/>
         </geometry>
       </collision>

File: src/kiwi_description/kiwi_drive_description/urdf/assemblies/wheel_2_link.urdf.xacro (robot description, xacro)
@@ -13,5 +13,5 @@
         <origin xyz="0.129426 -0.595834 0.367959" rpy="3.119159 -1.068867 1.618682"/>
         <geometry>
-          <mesh filename="package://Kiwi_Drive_Full_Assembly_Copy_Copy_description/meshes/wheel_2_link/wheel_2_link_Omni_Wheel.dae" scale="1 1 1"/>
+          <mesh filename="package://kiwi_drive_description/meshes/wheel_2_link/wheel_2_link_Omni_Wheel.dae" scale="1 1 1"/>
         </geometry>
         <material name="Steel"/>
@@ -20,5 +20,5 @@
         <origin xyz="0.129426 -0.595834 0.367959" rpy="3.119159 -1.068867 1.618682"/>
         <geometry>
-          <mesh filename="package://Kiwi_Drive_Full_Assembly_Copy_Copy_description/meshes/wheel_2_link/wheel_2_link_Omni_Wheel_collision.stl" scale="0.01 0.01 0.01"/>
+          <mesh filename="package://kiwi_drive_description/meshes/wheel_2_link/wheel_2_link_Omni_Wheel_collision.stl" scale="0.01 0.01 0.01"/>
         </geometry>
       </collision>

File: src/kiwi_description/kiwi_drive_description/urdf/assemblies/wheel_3_link.urdf.xacro (robot description, xacro)
@@ -13,5 +13,5 @@
         <origin xyz="-0.089816 0.603077 0.367959" rpy="3.119159 -1.068867 -1.588963"/>
         <geometry>
-          <mesh filename="package://Kiwi_Drive_Full_Assembly_Copy_Copy_description/meshes/wheel_3_link/wheel_3_link_Omni_Wheel.dae" scale="1 1 1"/>
+          <mesh filename="package://kiwi_drive_description/meshes/wheel_3_link/wheel_3_link_Omni_Wheel.dae" scale="1 1 1"/>
         </geometry>
         <material name="Steel"/>
@@ -20,5 +20,5 @@
         <origin xyz="-0.089816 0.603077 0.367959" rpy="3.119159 -1.068867 -1.588963"/>
         <geometry>
-          <mesh filename="package://Kiwi_Drive_Full_Assembly_Copy_Copy_description/meshes/wheel_3_link/wheel_3_link_Omni_Wheel_collision.stl" scale="0.01 0.01 0.01"/>
+          <mesh filename="package://kiwi_drive_description/meshes/wheel_3_link/wheel_3_link_Omni_Wheel_collision.stl" scale="0.01 0.01 0.01"/>
         </geometry>
       </collision>
