Commit message: Add physical SLAM and Nav2 bringup
Co-authored-by: Cursor <cursoragent@cursor.com>

File: src/kiwi_description/kiwi_drive_description/urdf/Kiwi_Drive_Full_Assembly_Copy_Copy.urdf.xacro (robot description, xacro)
@@ -1,4 +1,15 @@
 <?xml version="1.0"?>
 <robot xmlns:xacro="http://www.ros.org/wiki/xacro" name="Kiwi_Drive_Full_Assembly_Copy_Copy">
+  <!-- Physical bringup disables the generated ros2_control mock system. -->
+  <xacro:arg name="use_mock_hardware" default="true"/>
+  <!--
+    Provisional LD19 optical-frame pose relative to base_link.
+    These values preserve the existing field-tested patch transform and MUST
+    be physically measured and verified on the assembled robot.
+  -->
+  <xacro:arg name="laser_x" default="0.114"/>
+  <xacro:arg name="laser_y" default="0.0"/>
+  <xacro:arg name="laser_z" default="0.10977"/>
+  <xacro:arg name="laser_yaw" default="-1.5707963267948966"/>
   <!-- Materials (shared across all assemblies) -->
   <material name="Steel">
@@ -11,4 +22,5 @@
   <xacro:include filename="$(find kiwi_drive_description)/urdf/assemblies/wheel_3_link.urdf.xacro"/>
   <xacro:include filename="$(find kiwi_drive_description)/urdf/assemblies/lidar_link.urdf.xacro"/>
+  <xacro:include filename="$(find kiwi_drive_description)/urdf/assemblies/sensor_frames.urdf.xacro"/>
   <!-- Instantiate assemblies -->
   <xacro:base_link prefix=""/>
@@ -17,4 +29,11 @@
   <xacro:wheel_3_link prefix=""/>
   <xacro:lidar_link prefix=""/>
+  <xacro:kiwi_sensor_frames
+    prefix=""
+    parent="base_link"
+    laser_x="$(arg laser_x)"
+    laser_y="$(arg laser_y)"
+    laser_z="$(arg laser_z)"
+    laser_yaw="$(arg laser_yaw)"/>
   <!-- Mount joints (cross-assembly connections) -->
   <!-- These define how assemblies connect to each other. -->
@@ -48,38 +67,40 @@
     <origin xyz="-0.000151 -0.115009 0.024945" rpy="0.000000 0.000000 0.000000"/>
   </joint>
-  <!-- ROS 2 control: generated generic system -->
-  <ros2_control name="Kiwi_Drive_Full_Assembly_Copy_Copy_system" type="system">
-    <hardware>
-      <plugin>mock_components/GenericSystem</plugin>
-      <param name="cmd_topic">sim/Kiwi_Drive_Full_Assembly_Copy_Copy_system/cmd</param>
-      <param name="state_topic">sim/Kiwi_Drive_Full_Assembly_Copy_Copy_system/state</param>
-    </hardware>
-    <joint name="wheel_1_to_base_link">
-      <command_interface name="position"/>
-      <command_interface name="velocity"/>
-      <state_interface name="position">
-        <param name="initial_value">0.0</param>
-      </state_interface>
-      <state_interface name="velocity"/>
-      <state_interface name="effort"/>
-    </joint>
-    <joint name="wheel_2_to_base_link">
-      <command_interface name="position"/>
-      <command_interface name="velocity"/>
-      <state_interface name="position">
-        <param name="initial_value">0.0</param>
-      </state_interface>
-      <state_interface name="velocity"/>
-      <state_interface name="effort"/>
-    </joint>
-    <joint name="wheel_3_to_base_link">
-      <command_interface name="position"/>
-      <command_interface name="velocity"/>
-      <state_interface name="position">
-        <param name="initial_value">0.0</param>
-      </state_interface>
-      <state_interface name="velocity"/>
-      <state_interface name="effort"/>
-    </joint>
-  </ros2_control>
+  <xacro:if value="$(arg use_mock_hardware)">
+    <!-- Visualization-only generated generic system; never used by hardware.launch.py. -->
+    <ros2_control name="Kiwi_Drive_Full_Assembly_Copy_Copy_system" type="system">
+      <hardware>
+        <plugin>mock_components/GenericSystem</plugin>
+        <param name="cmd_topic">sim/Kiwi_Drive_Full_Assembly_Copy_Copy_system/cmd</param>
+        <param name="state_topic">sim/Kiwi_Drive_Full_Assembly_Copy_Copy_system/state</param>
+      </hardware>
+      <joint name="wheel_1_to_base_link">
+        <command_interface name="position"/>
+        <command_interface name="velocity"/>
+        <state_interface name="position">
+          <param name="initial_value">0.0</param>
+        </state_interface>
+        <state_interface name="velocity"/>
+        <state_interface name="effort"/>
+      </joint>
+      <joint name="wheel_2_to_base_link">
+        <command_interface name="position"/>
+        <command_interface name="velocity"/>
+        <state_interface name="position">
+          <param name="initial_value">0.0</param>
+        </state_interface>
+        <state_interface name="velocity"/>
+        <state_interface name="effort"/>
+      </joint>
+      <joint name="wheel_3_to_base_link">
+        <command_interface name="position"/>
+        <command_interface name="velocity"/>
+        <state_interface name="position">
+          <param name="initial_value">0.0</param>
+        </state_interface>
+        <state_interface name="velocity"/>
+        <state_interface name="effort"/>
+      </joint>
+    </ros2_control>
+  </xacro:if>
 </robot>

Commit message: Align CAD visuals with ROS forward and publish wheel joint zeros.
The Fusion chassis sat 90 degrees to the right of base_link, so the lidar mesh was on the robot's right while the scan was in front. Rotate CAD mounts and the base mesh, and publish dummy wheel states so RViz can draw the omni wheels.

Co-authored-by: Cursor <cursoragent@cursor.com>

File: src/kiwi_description/kiwi_drive_description/urdf/Kiwi_Drive_Full_Assembly_Copy_Copy.urdf.xacro (robot description, xacro)
@@ -41,8 +41,13 @@
   <!-- update the include + macro call above, and adjust -->
   <!-- parent/child link names in the mount joint below. -->
+  <!--
+    CAD mount poses are yawed +90 deg about Z so Fusion chassis front
+    (lidar plate) lands on ROS +X. Do not change base_laser; that optical
+    frame is already REP-103.
+  -->
   <joint name="wheel_1_to_base_link" type="continuous">
     <parent link="base_link"/>
     <child link="wheel_1_link_Omni_Wheel"/>
-    <origin xyz="0.269094 -0.155140 -0.028295" rpy="-1.588336 0.031105 1.057255"/>
+    <origin xyz="0.155140 0.269094 -0.028295" rpy="-1.588336 0.031105 2.628051"/>
     <axis xyz="0.000000 0.000000 1.000000"/>
     <limit effort="100.0" velocity="1.00"/>
@@ -51,5 +56,5 @@
     <parent link="base_link"/>
     <child link="wheel_2_link_Omni_Wheel"/>
-    <origin xyz="-0.000532 0.310563 -0.028788" rpy="1.574419 -0.000039 0.010768"/>
+    <origin xyz="-0.310563 -0.000532 -0.028788" rpy="1.574419 -0.000039 1.581564"/>
     <axis xyz="0.000000 0.000000 1.000000"/>
     <limit effort="100.0" velocity="1.00"/>
@@ -58,5 +63,5 @@
     <parent link="base_link"/>
     <child link="wheel_3_link_Omni_Wheel"/>
-    <origin xyz="-0.269016 -0.155795 -0.029665" rpy="-1.549628 0.035717 -1.035628"/>
+    <origin xyz="0.155795 -0.269016 -0.029665" rpy="-1.549628 0.035717 0.535168"/>
     <axis xyz="0.000000 0.000000 1.000000"/>
     <limit effort="100.0" velocity="1.00"/>
@@ -65,5 +70,5 @@
     <parent link="base_link"/>
     <child link="Lidar_Mounting_Plate"/>
-    <origin xyz="-0.000151 -0.115009 0.024945" rpy="0.000000 0.000000 0.000000"/>
+    <origin xyz="0.115009 -0.000151 0.024945" rpy="0.000000 0.000000 1.570796"/>
   </joint>
   <xacro:if value="$(arg use_mock_hardware)">

File: src/kiwi_description/kiwi_drive_description/urdf/assemblies/base_link.urdf.xacro (robot description, xacro)
@@ -11,5 +11,6 @@
       </inertial>
       <visual>
-        <origin xyz="0.000000 0.000000 0.000000" rpy="0.000000 0.000000 -2.094395"/>
+        <!-- Extra +90 deg yaw: Fusion chassis front was on ROS -Y (right). -->
+        <origin xyz="0.000000 0.000000 0.000000" rpy="0.000000 0.000000 -0.523599"/>
         <geometry>
           <mesh filename="package://kiwi_drive_description/meshes/base_link/base_link.dae" scale="1 1 1"/>
@@ -18,5 +19,5 @@
       </visual>
       <collision>
-        <origin xyz="0.000000 0.000000 0.000000" rpy="0.000000 0.000000 -2.094395"/>
+        <origin xyz="0.000000 0.000000 0.000000" rpy="0.000000 0.000000 -0.523599"/>
         <geometry>
           <mesh filename="package://kiwi_drive_description/meshes/base_link/base_link_collision.stl" scale="0.01 0.01 0.01"/>
